File: small/Apple II Prototype.kicad_pcb (KiCad board)
At the start: 2 copper layers, 99.7 x 78.7 mm, 40 parts, among them J1 Breakout, P1 Prototype_26, P10 Prototype_23, P11 Prototype_23, P12 Prototype_23, P13 Prototype_23, P14 Prototype_23, P15 Prototype_23, P16 Prototype_23, P17 Prototype_23, P18 Prototype_23, P19 Prototype_23, P2 Prototype_26, P20 Prototype_23, P21 Prototype_23, P22 Prototype_23, P23 Prototype_23, P24 Prototype_23, P25 Prototype_23, P26 Prototype_23, P27 Prototype_23, P28 Prototype_23, P29 Prototype_23, P3 Prototype_26, P30 Prototype_23, P31 Prototype_23, P32 Prototype_23, P33 Prototype_23, P34 Prototype_23, P35 Prototype_23, P36 Prototype_26, P37 Prototype_26, P38 Prototype_26, P4 Prototype_26, P5 Prototype_26, P6 Prototype_26, P7 Prototype_26, P8 Prototype_26, P9 Prototype_23

Commit message: Added fullsize board and signal names to boards
Connections:
- net /~M2SEL renamed /~USER1
- BUS1 pad 19: (no net) -> /SYNC
- BUS1 pad 35: (no net) -> /COLOR_REF
- J1 pad 19: (no net) -> /SYNC
- J1 pad 35: (no net) -> /COLOR_REF
Routing:
- net /COLOR_REF: track 0.00 -> 11.8 mm
- net /SYNC: track 0.00 -> 8.25 mm
Other:
- board text removed: "+12v"
- board text removed: "+5V"
- board text removed: "A0"
- board text removed: "A15"
- board text removed: "D0"
- board text removed: "D7"
- board text removed: "GND"
- board text removed: "I/O SEL"
- board text removed: "R/W"
- board text removed: "STROBE"
- board text removed: "~RESET"
- board text removed: "Ø0"
- board text removed: "Ø1"
