File: small/Apple II Prototype.sch (KiCad schematic (older format))
At the start: 40 parts, among them J1 Breakout, P1 Prototype_26, P10 Prototype_23, P11 Prototype_23, P12 Prototype_23, P13 Prototype_23, P14 Prototype_23, P15 Prototype_23, P16 Prototype_23, P17 Prototype_23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

Commit message: Added fullsize board and signal names to boards
Connections:
- net SYNC: now reaches BUS1.19 (n.c.)
- net SYNC: now also J1.19 (Pin_19)
- net COLOR_REF: now reaches BUS1.35 (n.c.)
- net COLOR_REF: now also J1.35 (Pin_35)
- net ~M2SEL renamed ~USER1
- no-connect marks 2 -> 0
